Commit message: bugfix: including right inertia and adding init rviz config

File: src/robot_description/urdf/robot_base.xacro (robot description, xacro)
@@ -19,29 +19,47 @@
         <xacro:box_inertia m="5.0" l="${base_length}" w="${base_width}" h="${base_height}"
                            xyz="0 0 ${base_height / 2.0 + wheel_radius}" rpy="0 0 0" />
+        <collision>
+            <geometry>
+                <box size="${base_length} ${base_width} ${base_height}" />
+            </geometry>
+            <origin xyz="0 0 ${base_height / 2.0 + wheel_radius}" rpy="0 0 0" />
+        </collision>
     </link>
   <xacro:macro name="throttle_wheel_link" params="prefix">
       <link name="${prefix}_throttle_wheel_link">
-          <visual>
-              <geometry>
-                  <cylinder radius="${wheel_radius}" length="${wheel_length}" />
-              </geometry>
-              <origin xyz="0 0 0" rpy="${pi / 2.0} 0 0" />
-              <material name="blue" />
-          </visual>
-          <xacro:cylinder_inertia m="1.0" r="${wheel_radius}" h="${wheel_length}"
-                                  xyz="0 0 0" rpy="${pi / 2.0} 0 0" />
+        <visual>
+            <geometry>
+                <cylinder radius="${wheel_radius}" length="${wheel_length}" />
+            </geometry>
+            <origin xyz="0 0 0" rpy="${pi / 2.0} 0 0" />
+            <material name="blue" />
+        </visual>
+        <xacro:cylinder_inertia m="1.0" r="${wheel_radius}" h="${wheel_length}"
+                                xyz="0 0 0" rpy="${pi / 2.0} 0 0" />
+        <collision>
+            <geometry>
+                <cylinder radius="${wheel_radius}" length="${wheel_length}" />
+            </geometry>
+            <origin xyz="0 0 0" rpy="${pi / 2.0} 0 0" />
+        </collision>
       </link>
   </xacro:macro>
   <xacro:macro name="steering_wheel_link" params="prefix">
       <link name="${prefix}_steering_wheel_link">
-          <visual>
-              <geometry>
-                  <cylinder radius="${wheel_radius/10}" length="${wheel_length/10}" />
-              </geometry>
-              <origin xyz="0 0 0" rpy="${pi / 2.0} 0 0" />
-              <material name="gray" />
-          </visual>
-          <xacro:cylinder_inertia m="1.0" r="${wheel_radius}" h="${wheel_length}"
-                                  xyz="0 0 0" rpy="${pi / 2.0} 0 0" />
+        <visual>
+            <geometry>
+                <cylinder radius="${wheel_radius/10}" length="${wheel_length/10}" />
+            </geometry>
+            <origin xyz="0 0 0" rpy="${pi / 2.0} 0 0" />
+            <material name="gray" />
+        </visual>
+        <xacro:cylinder_inertia m="1.0" r="${wheel_radius}" h="${wheel_length}"
+                                xyz="0 0 0" rpy="${pi / 2.0} 0 0" />
+        <collision>
+            <geometry>
+                <cylinder radius="${wheel_radius/10}" length="${wheel_length/10}" />
+            </geometry>
+            <origin xyz="0 0 0" rpy="${pi / 2.0} 0 0" />
+        </collision>
       </link>
   </xacro:macro>

File: src/robot_description/urdf/sensors.xacro (robot description, xacro)
@@ -9,4 +9,12 @@
       <material name="white"/>
     </visual>
+    <xacro:cylinder_inertia m="0.2" r="${lidar_size / 2.0}" h="${lidar_size}"
+                            xyz="0 0 0" rpy="0 0 0" />
+    <collision>
+        <geometry>
+          <cylinder length="${lidar_size}" radius="${lidar_size / 2.0}"/>
+        </geometry>
+      <origin xyz="0 0 0" rpy="0 0 0"/>
+    </collision>
   </link>
   <link name="camera">
@@ -18,4 +26,12 @@
       <material name="white"/>
     </visual>
+    <xacro:box_inertia m="0.3" l="${camera_size / 4.0}" w="${camera_size}" h="${camera_size / 4.0}"
+                        xyz="0 0 0" rpy="0 0 0" />
+    <collision>
+        <geometry>
+          <box size="${camera_size / 4.0} ${camera_size} ${camera_size / 4.0}"/>
+        </geometry>
+      <origin xyz="0 0 0" rpy="0 0 0"/>
+    </collision>
   </link>
   <joint name="joint_camera" type="fixed">
